Commit message: Big balls

File: src/rhex_ws/rhex_description/urdf/macros.xacro (robot description, xacro)
@@ -4,5 +4,5 @@
       <visual>
         <geometry>
-          <mesh filename="$(find rhex_description)/meshes/${mesh}" scale="${scale}"/>
+          <mesh filename="package://rhex_description/urdf/meshes/${mesh}" scale="${scale}"/>
         </geometry>
         <material name="white"/>
@@ -10,5 +10,5 @@
       <collision>
         <geometry>
-          <mesh filename="$(find rhex_description)/meshes/${mesh}" scale="${scale}"/>
+          <mesh filename="package://rhex_description/urdf/meshes/${mesh}" scale="${scale}"/>
         </geometry>
       </collision>

File: src/rhex_ws/rhex_description/urdf/rhex.control.xacro (robot description, xacro)
@@ -7,5 +7,5 @@
           <plugin>gazebo_ros2_control/GazeboSystem</plugin>
         </hardware>
-        <xacro:include filename="$(find rhex_description)/urdf/joints_interfaces.xacro"/>
+        <xacro:include filename="package://rhex_description/urdf/joints_interfaces.xacro"/>
       </ros2_control>
     </xacro:if>
@@ -15,5 +15,5 @@
           <plugin>giga_hw_interface/GigaHardwareInterface</plugin>
         </hardware>
-        <xacro:include filename="$(find rhex_description)/urdf/joints_interfaces.xacro"/>
+        <xacro:include filename="package://rhex_description/urdf/joints_interfaces.xacro"/>
       </ros2_control>
     </xacro:unless>

File: src/rhex_ws/rhex_description/urdf/rhex.xacro (robot description, xacro)
@@ -14,5 +14,5 @@
     <visual>
       <geometry>
-        <mesh filename="$(find rhex_description)/meshes/Chassis.stl" scale="${scale}"/>
+        <mesh filename="package://rhex_description/urdf/meshes/Chassis.stl" scale="${scale}"/>
       </geometry>
       <material name="ibm_blue"/>
@@ -20,5 +20,5 @@
     <collision>
       <geometry>
-        <mesh filename="$(find rhex_description)/meshes/Chassis.stl" scale="${scale}"/>
+        <mesh filename="package://rhex_description/urdf/meshes/Chassis.stl" scale="${scale}"/>
       </geometry>
     </collision>
@@ -33,5 +33,5 @@
     <origin xyz="0 0 0" rpy="0 0 0"/>
     <geometry>
-      <mesh filename="$(find rhex_description)/meshes/lidar.stl" scale="1 1 1"/>
+      <mesh filename="package://rhex_description/urdf/meshes/lidar.stl" scale="1 1 1"/>
     </geometry>
     <material name="gray"/>
@@ -52,5 +52,5 @@
     <origin xyz="0 0 0" rpy="0 0 0"/>
     <geometry>
-      <mesh filename="$(find rhex_description)/meshes/stereo_camera.stl" scale="1 1 1"/>
+      <mesh filename="package://rhex_description/urdf/meshes/stereo_camera.stl" scale="1 1 1"/>
     </geometry>
     <material name="gray"/>
@@ -71,5 +71,5 @@
     <origin xyz="0 0 0" rpy="0 0 0"/>
     <geometry>
-      <mesh filename="$(find rhex_description)/meshes/thermal_camera.stl" scale="1 1 1"/>
+      <mesh filename="package://rhex_description/urdf/meshes/thermal_camera.stl" scale="1 1 1"/>
     </geometry>
     <material name="gray"/>

Commit message: a

File: src/rhex_ws/rhex_description/urdf/macros.xacro (robot description, xacro)
@@ -4,5 +4,5 @@
       <visual>
         <geometry>
-          <mesh filename="package://rhex_description/urdf/meshes/${mesh}" scale="${scale}"/>
+          <mesh filename="$(find rhex_description)/meshes/${mesh}" scale="${scale}"/>
         </geometry>
         <material name="white"/>
@@ -10,5 +10,5 @@
       <collision>
         <geometry>
-          <mesh filename="package://rhex_description/urdf/meshes/${mesh}" scale="${scale}"/>
+          <mesh filename="$(find rhex_description)/meshes/${mesh}" scale="${scale}"/>
         </geometry>
       </collision>

File: src/rhex_ws/rhex_description/urdf/rhex.xacro (robot description, xacro)
@@ -14,5 +14,5 @@
     <visual>
       <geometry>
-        <mesh filename="package://rhex_description/urdf/meshes/Chassis.stl" scale="${scale}"/>
+        <mesh filename="$(find rhex_description)/meshes/Chassis.stl" scale="${scale}"/>
       </geometry>
       <material name="ibm_blue"/>
@@ -20,5 +20,5 @@
     <collision>
       <geometry>
-        <mesh filename="package://rhex_description/urdf/meshes/Chassis.stl" scale="${scale}"/>
+        <mesh filename="$(find rhex_description)/meshes/Chassis.stl" scale="${scale}"/>
       </geometry>
     </collision>
@@ -33,5 +33,5 @@
     <origin xyz="0 0 0" rpy="0 0 0"/>
     <geometry>
-      <mesh filename="package://rhex_description/urdf/meshes/lidar.stl" scale="1 1 1"/>
+      <mesh filename="$(find rhex_description)/meshes/lidar.stl" scale="1 1 1"/>
     </geometry>
     <material name="gray"/>
@@ -52,5 +52,5 @@
     <origin xyz="0 0 0" rpy="0 0 0"/>
     <geometry>
-      <mesh filename="package://rhex_description/urdf/meshes/stereo_camera.stl" scale="1 1 1"/>
+      <mesh filename="$(find rhex_description)/meshes/stereo_camera.stl" scale="1 1 1"/>
     </geometry>
     <material name="gray"/>
@@ -71,5 +71,5 @@
     <origin xyz="0 0 0" rpy="0 0 0"/>
     <geometry>
-      <mesh filename="package://rhex_description/urdf/meshes/thermal_camera.stl" scale="1 1 1"/>
+      <mesh filename="$(find rhex_description)/meshes/thermal_camera.stl" scale="1 1 1"/>
     </geometry>
     <material name="gray"/>

Commit message: rs update

File: src/rhex_ws/rhex_description/urdf/macros.xacro (robot description, xacro)
@@ -4,5 +4,5 @@
       <visual>
         <geometry>
-          <mesh filename="$(find rhex_description)/meshes/${mesh}" scale="${scale}"/>
+          <mesh filename="package:/rhex_ws/rhex_description/meshes/${mesh}" scale="${scale}"/>
         </geometry>
         <material name="white"/>
@@ -10,5 +10,5 @@
       <collision>
         <geometry>
-          <mesh filename="$(find rhex_description)/meshes/${mesh}" scale="${scale}"/>
+          <mesh filename="package:/rhex_ws/rhex_description/meshes/${mesh}" scale="${scale}"/>
         </geometry>
       </collision>

File: src/rhex_ws/rhex_description/urdf/rhex.xacro (robot description, xacro)
@@ -14,5 +14,5 @@
     <visual>
       <geometry>
-        <mesh filename="$(find rhex_description)/meshes/Chassis.stl" scale="${scale}"/>
+        <mesh filename="package:/rhex_ws/rhex_description/meshes/Chassis.stl" scale="${scale}"/>
       </geometry>
       <material name="ibm_blue"/>
@@ -20,5 +20,5 @@
     <collision>
       <geometry>
-        <mesh filename="$(find rhex_description)/meshes/Chassis.stl" scale="${scale}"/>
+        <mesh filename="package:/rhex_ws/rhex_description/Chassis.stl" scale="${scale}"/>
       </geometry>
     </collision>
@@ -33,5 +33,5 @@
     <origin xyz="0 0 0" rpy="0 0 0"/>
     <geometry>
-      <mesh filename="$(find rhex_description)/meshes/lidar.stl" scale="1 1 1"/>
+      <mesh filename="package:/rhex_ws/rhex_description/meshes/lidar.stl" scale="1 1 1"/>
     </geometry>
     <material name="gray"/>
@@ -52,5 +52,5 @@
     <origin xyz="0 0 0" rpy="0 0 0"/>
     <geometry>
-      <mesh filename="$(find rhex_description)/meshes/stereo_camera.stl" scale="1 1 1"/>
+      <mesh filename="package:/rhex_ws/rhex_description/meshes/stereo_camera.stl" scale="1 1 1"/>
     </geometry>
     <material name="gray"/>
@@ -71,5 +71,5 @@
     <origin xyz="0 0 0" rpy="0 0 0"/>
     <geometry>
-      <mesh filename="$(find rhex_description)/meshes/thermal_camera.stl" scale="1 1 1"/>
+      <mesh filename="package:/rhex_ws/rhex_description/meshes/thermal_camera.stl" scale="1 1 1"/>
     </geometry>
     <material name="gray"/>

Commit message: in prog

File: src/rhex_ws/rhex_description/urdf/macros.xacro (robot description, xacro)
@@ -4,5 +4,5 @@
       <visual>
         <geometry>
-          <mesh filename="package:/rhex_ws/rhex_description/meshes/${mesh}" scale="${scale}"/>
+          <mesh filename="$(find rhex_description)/meshes/${mesh}" scale="${scale}"/>
         </geometry>
         <material name="white"/>
@@ -10,5 +10,5 @@
       <collision>
         <geometry>
-          <mesh filename="package:/rhex_ws/rhex_description/meshes/${mesh}" scale="${scale}"/>
+          <mesh filename="$(find rhex_description)/meshes/${mesh}" scale="${scale}"/>
         </geometry>
       </collision>

File: src/rhex_ws/rhex_description/urdf/rhex.xacro (robot description, xacro)
@@ -14,5 +14,5 @@
     <visual>
       <geometry>
-        <mesh filename="package:/rhex_ws/rhex_description/meshes/Chassis.stl" scale="${scale}"/>
+        <mesh filename="$(find rhex_description)/meshes/Chassis.stl" scale="${scale}"/>
       </geometry>
       <material name="ibm_blue"/>
@@ -20,5 +20,5 @@
     <collision>
       <geometry>
-        <mesh filename="package:/rhex_ws/rhex_description/Chassis.stl" scale="${scale}"/>
+        <mesh filename="$(find rhex_description)/meshes/Chassis.stl" scale="${scale}"/>
       </geometry>
     </collision>
@@ -33,5 +33,5 @@
     <origin xyz="0 0 0" rpy="0 0 0"/>
     <geometry>
-      <mesh filename="package:/rhex_ws/rhex_description/meshes/lidar.stl" scale="1 1 1"/>
+      <mesh filename="$(find rhex_description)/meshes/lidar.stl" scale="1 1 1"/>
     </geometry>
     <material name="gray"/>
@@ -52,5 +52,5 @@
     <origin xyz="0 0 0" rpy="0 0 0"/>
     <geometry>
-      <mesh filename="package:/rhex_ws/rhex_description/meshes/stereo_camera.stl" scale="1 1 1"/>
+      <mesh filename="$(find rhex_description)/meshes/stereo_camera.stl" scale="1 1 1"/>
     </geometry>
     <material name="gray"/>
@@ -71,5 +71,5 @@
     <origin xyz="0 0 0" rpy="0 0 0"/>
     <geometry>
-      <mesh filename="package:/rhex_ws/rhex_description/meshes/thermal_camera.stl" scale="1 1 1"/>
+      <mesh filename="$(find rhex_description)/meshes/thermal_camera.stl" scale="1 1 1"/>
     </geometry>
     <material name="gray"/>

Commit message: new test

File: src/rhex_ws/rhex_description/urdf/macros.xacro (robot description, xacro)
@@ -29,5 +29,5 @@
       <origin xyz="${xyz}" rpy="0 0 0"/>
       <axis xyz="1 0 0"/>
-      <limit effort="30" velocity="4"/>
+      <limit effort="10" velocity="5.0"/>
       <dynamics damping="1.0" friction="1.0"/>\
     </joint>

File: src/rhex_ws/rhex_description/urdf/rhex.control.xacro (robot description, xacro)
@@ -1,5 +1,5 @@
 <?xml version="1.0"?>
 <robot xmlns:xacro="http://www.ros.org/wiki/xacro">
-  <xacro:macro name="rhex_control" params="use_sim:=false">
+  <xacro:macro name="rhex_control" params="use_sim:=true">
     <xacro:if value="${use_sim}">
       <ros2_control name="RHexHardware" type="system">

File: src/rhex_ws/rhex_description/urdf/rhex.xacro (robot description, xacro)
@@ -24,5 +24,5 @@
     </collision>
     <inertial>
-      <mass value="1.5"/>
+      <mass value="4"/>
       <origin xyz="0 0 0.05"/>
       <inertia ixx="2.222e-2" ixy="4.654e-6" ixz="1.02836e-5" iyy="1.129e-2" iyz="4.82214e-5" izz="2.96e-2"/>
